File: Industrial_IoT_Controller.kicad_pcb (KiCad board)
At the start: 4 copper layers, 102 x 87 mm, 72 parts, among them J1 Screw_Terminal_01x02, J2 Screw_Terminal_01x02, J3 Screw_Terminal_01x02, J4 Screw_Terminal_01x02, J5 RLY PIN, K1 JQC-3FF/024-1ZS(551)_C2976878, Q1 TSM2309, Q2 MMBT3904, Q3 MMBT3904, Q4 BSS138, U1 LM2596S-5, U2 TLV76733DRVx, U3 ESP32-WROOM-32E, U4 MAX485E, U5 CP2102N-Axx-xQFN24

Commit message: Final Schematic
Parts:
- removed RESET1: RESET, Button_Switch_THT:SW_PUSH_6mm
- added C15: 100nF, lcsc_footprints:C1591_C0603, F.Cu at (151.6, 100.0)
- added C16: 100nF, lcsc_footprints:C1591_C0603, F.Cu at (155.6, 86.7)
- added C17: 4.7uF, lcsc_footprints:C1779_C0805, F.Cu at (157.2, 121.1)
- added C18: 100nF, lcsc_footprints:C1590_C0603, F.Cu at (155.6, 93.5)
- added C19: 10nF, lcsc_footprints:C100042_C0603, F.Cu at (155.6, 96.2)
- added C20: 100nF, lcsc_footprints:C1591_C0603, F.Cu at (155.6, 94.7)
- added C21: 100nF, lcsc_footprints:C1591_C0603, F.Cu at (155.6, 97.3)
- added C22: 100nF, lcsc_footprints:C1590_C0603, F.Cu at (155.6, 104.2)
- added C23: 10uF, lcsc_footprints:C85713_C0603, F.Cu at (159.6, 90.8)
- added C24: 10uF, lcsc_footprints:C440198_C0805, F.Cu at (157.2, 124.0)
- added C25: 100nF, lcsc_footprints:C1591_C0603, F.Cu at (159.6, 89.3)
- added C26: 10uF, lcsc_footprints:C440198_C0805, F.Cu at (157.2, 127.0)
- added C27: 100nF, lcsc_footprints:C1591_C0603, F.Cu at (159.6, 92.0)
- added C28: 10uF, lcsc_footprints:C440198_C0805, F.Cu at (162.2, 115.2)
- added C29: 100nF, lcsc_footprints:C1591_C0603, F.Cu at (159.6, 94.7)
- added C30: 100nF, lcsc_footprints:C1590_C0603, F.Cu at (159.6, 101.5)
- added C31: 10uF, lcsc_footprints:C85713_C0603, F.Cu at (159.6, 104.2)
- added C32: 100nF, lcsc_footprints:C1590_C0603, F.Cu at (163.6, 90.8)
- added C33: 10nF, lcsc_footprints:C100042_C0603, F.Cu at (163.6, 93.5)
- added C34: 10uF, lcsc_footprints:C440198_C0805, F.Cu at (162.2, 118.1)
- added C35: 100nF, lcsc_footprints:C1591_C0603, F.Cu at (163.7, 92.0)
- added C36: 10uF, lcsc_footprints:C440198_C0805, F.Cu at (162.2, 121.1)
- added C37: 100nF, lcsc_footprints:C1591_C0603, F.Cu at (163.7, 94.7)
- added C38: 10uF, lcsc_footprints:C440198_C0805, F.Cu at (162.2, 124.0)
- added C39: 100nF, lcsc_footprints:C1591_C0603, F.Cu at (163.7, 97.3)
- added D14: BAT54JFILM, lcsc_footprints:C86299_SOD-323_L1_8-W1_3-LS2_5-RD, F.Cu at (190.9, 93.3)
- added D15: 1N4148W, lcsc_footprints:C917030_SOD-123_L2_8-W1_8-LS3_7-RD-1, F.Cu at (138.3, 117.7)
- added D16: SMBJ33A, lcsc_footprints:C353366_SMB_L4_4-W3_6-LS5_3-RD, F.Cu at (186.2, 81.1)
- added D17: BAT54JFILM, lcsc_footprints:C86299_SOD-323_L1_8-W1_3-LS2_5-RD, F.Cu at (190.9, 95.9)
- added D18: SMAJ5.0A, lcsc_footprints:C83329_SMA_L4_3-W2_6-LS5_2-RD, F.Cu at (144.7, 113.6)
- added D19: SMBJ12A, lcsc_footprints:C50087775_SMB_L4_6-W3_6-LS5_3-RD, F.Cu at (139.6, 130.5)
- added D20: SS14, lcsc_footprints:C2480_SMA_L4_2-W2_6-LS5_0-RD_1, F.Cu at (170.5, 116.5)
- added D21: SS14, lcsc_footprints:C2480_SMA_L4_2-W2_6-LS5_0-RD_1, F.Cu at (170.5, 120.3)
- added D22: SS14, lcsc_footprints:C2480_SMA_L4_2-W2_6-LS5_0-RD_1, F.Cu at (170.5, 124.2)
- added D23: SM712, Package_TO_SOT_SMD:SOT-23, F.Cu at (186.1, 137.8)
- added D24: SS14, lcsc_footprints:C2480_SMA_L4_2-W2_6-LS5_0-RD_1, F.Cu at (170.5, 128.0)
- added D25: SS14, lcsc_footprints:C2480_SMA_L4_2-W2_6-LS5_0-RD_1, F.Cu at (170.5, 131.9)
- added D26: SS14, lcsc_footprints:C2480_SMA_L4_2-W2_6-LS5_0-RD_1, F.Cu at (170.5, 135.7)
- added F2: 500 mA, lcsc_footprints:C163512_F1206, B.Cu at (169.5, 117.2)
- added F3: SMD0805-010-60V, lcsc_footprints:C6851463_F0805, F.Cu at (186.3, 102.9)
- added F4: SMD0805-010-60V, lcsc_footprints:C6851463_F0805, F.Cu at (186.3, 106.1)
- added F5: SMD0805-010-60V, lcsc_footprints:C6851463_F0805, F.Cu at (186.3, 109.3)
- added F6: SMD0805-010-60V, lcsc_footprints:C6851463_F0805, F.Cu at (186.3, 112.5)
- added J10: RLY PIN, TerminalBlock_Phoenix:TerminalBlock_Phoenix_MKDS-3-3-5.08_1x03_P5.08mm_Horizontal, F.Cu at (116.2, 71.2)
- added J12: RLY PIN, TerminalBlock_Phoenix:TerminalBlock_Phoenix_MKDS-3-3-5.08_1x03_P5.08mm_Horizontal, F.Cu at (116.1, 88.8)
- added J13: RLY PIN, TerminalBlock_Phoenix:TerminalBlock_Phoenix_MKDS-3-3-5.08_1x03_P5.08mm_Horizontal, F.Cu at (116.2, 98.2)
- added J14: RLY PIN, TerminalBlock_Phoenix:TerminalBlock_Phoenix_MKDS-3-3-5.08_1x03_P5.08mm_Horizontal, F.Cu at (116.2, 111.7)
- added J15: RLY PIN, TerminalBlock_Phoenix:TerminalBlock_Phoenix_MKDS-3-3-5.08_1x03_P5.08mm_Horizontal, F.Cu at (116.2, 125.2)
- added J6: Screw_Terminal_01x02, TerminalBlock_Phoenix:TerminalBlock_Phoenix_MKDS-3-2-5.08_1x02_P5.08mm_Horizontal, F.Cu at (145.7, 57.6)
- added J7: Screw_Terminal_01x02, TerminalBlock_Phoenix:TerminalBlock_Phoenix_MKDS-3-2-5.08_1x02_P5.08mm_Horizontal, F.Cu at (157.9, 57.6)
- added J8: RLY PIN, TerminalBlock_Phoenix:TerminalBlock_Phoenix_MKDS-3-3-5.08_1x03_P5.08mm_Horizontal, F.Cu at (116.2, 44.1)
- added J9: RLY PIN, TerminalBlock_Phoenix:TerminalBlock_Phoenix_MKDS-3-3-5.08_1x03_P5.08mm_Horizontal, F.Cu at (116.2, 57.6)
- added JP1: RS485_TERM, lcsc_footprints:C32713268_HDR-TH_2P-P2_54-V-M-3, F.Cu at (162.5, 139.3)
- added K2: JQC-3FF/024-1ZS(551)_C2976878, lcsc_footprints:C2976878_RELAY-TH_HF_JQC-3FF, F.Cu at (101.5, 62.2)
- added K3: JQC-3FF/024-1ZS(551)_C2976878, lcsc_footprints:C2976878_RELAY-TH_HF_JQC-3FF, F.Cu at (101.5, 78.8)
- added K4: JQC-3FF/024-1ZS(551)_C2976878, lcsc_footprints:C2976878_RELAY-TH_HF_JQC-3FF, F.Cu at (101.5, 95.5)
- added K5: JQC-3FF/024-1ZS(551)_C2976878, lcsc_footprints:C2976878_RELAY-TH_HF_JQC-3FF, F.Cu at (101.5, 112.1)
- added K6: JQC-3FF/024-1ZS(551)_C2976878, lcsc_footprints:C2976878_RELAY-TH_HF_JQC-3FF, F.Cu at (101.5, 128.8)
- added L2: 2.2 uH, lcsc_footprints:C53198556_IND-SMD_L4_1-W4_1_ASFPIG4020, F.Cu at (186.1, 94.7)
- added L3: 600Ω±25% @100MHz, lcsc_footprints:C85833_L0603, F.Cu at (190.9, 106.7)
- added L4: 600Ω±25% @100MHz, lcsc_footprints:C85833_L0603, F.Cu at (190.9, 109.2)
- added LED1: 0805, lcsc_footprints:C2296_LED0805-R-RD, F.Cu at (170.1, 103.0)
- added LED2: 0805, lcsc_footprints:C2296_LED0805-R-RD, F.Cu at (170.1, 106.3)
- added LED3: YLED0805R, lcsc_footprints:C19171391_LED0805-R-RD_RED, F.Cu at (170.1, 109.6)
- added LED4: XL-2012UBC, lcsc_footprints:C965817_LED0805-RD, B.Cu at (167.2, 129.6)
- added LED5: 0805, lcsc_footprints:C2296_LED0805-R-RD, F.Cu at (170.1, 112.9)
- added LED6: 0805, lcsc_footprints:C2296_LED0805-R-RD, F.Cu at (175.6, 103.0)
- added LED7: XL-2012UBC, lcsc_footprints:C965817_LED0805-RD, F.Cu at (146.2, 132.8)
- added LED8: 0805, lcsc_footprints:C2296_LED0805-R-RD, F.Cu at (175.6, 106.3)
- added Q5: BSS138, lcsc_footprints:C52895_SOT-23-3_L2_9-W1_6-P1_90-LS2_8-BR, F.Cu at (186.0, 125.1)
- added Q6: BSS138, lcsc_footprints:C52895_SOT-23-3_L2_9-W1_6-P1_90-LS2_8-BR, F.Cu at (186.0, 129.4)
- added Q7: BSS138, lcsc_footprints:C52895_SOT-23-3_L2_9-W1_6-P1_90-LS2_8-BR, F.Cu at (190.5, 116.7)
- added Q8: BSS138, lcsc_footprints:C52895_SOT-23-3_L2_9-W1_6-P1_90-LS2_8-BR, F.Cu at (190.5, 120.9)
- added Q9: BSS138, lcsc_footprints:C52895_SOT-23-3_L2_9-W1_6-P1_90-LS2_8-BR, F.Cu at (190.5, 125.1)
- added R26: 1KΩ, lcsc_footprints:C22548_R0603, F.Cu at (135.8, 96.4)
- added R27: 4.7 kΩ, lcsc_footprints:C99782_R0603, F.Cu at (135.8, 98.9)
- added R28: 2.2 kΩ, lcsc_footprints:C525570_R1206, F.Cu at (132.8, 132.4)
- added R29: 2.2 kΩ, lcsc_footprints:C525570_R1206, F.Cu at (132.8, 135.7)
- added R30: 1KΩ, lcsc_footprints:C22548_R0603, F.Cu at (135.8, 101.4)
- added R31: 22.1KΩ, lcsc_footprints:C2960862_R0603, F.Cu at (135.8, 103.9)
- added R32: 47.KΩ, lcsc_footprints:C403243_R0603, F.Cu at (135.8, 106.3)
- added R33: 1KΩ, lcsc_footprints:C22548_R0603, F.Cu at (139.7, 86.6)
- added R34: 10KΩ, lcsc_footprints:C98220_R0603, F.Cu at (139.7, 89.0)
- added R35: 20KΩ, lcsc_footprints:C2907011_R0603, F.Cu at (139.7, 91.5)
- added R36: 150Ω, lcsc_footprints:C7065937_R0805, F.Cu at (145.8, 135.8)
- added R37: 1KΩ, lcsc_footprints:C22548_R0603, F.Cu at (139.7, 94.0)
- added R38: 10KΩ, lcsc_footprints:C98220_R0603, F.Cu at (139.7, 96.4)
- added R39: 100Ω, lcsc_footprints:C2906981_R0603, F.Cu at (139.7, 98.9)
- added R40: 100Ω, lcsc_footprints:C2906981_R0603, F.Cu at (139.7, 101.4)
- added R41: 100Ω, lcsc_footprints:C2906981_R0603, F.Cu at (139.7, 103.9)
- added R42: 1KΩ, lcsc_footprints:C22548_R0603, F.Cu at (139.7, 106.3)
- added R43: 10KΩ, lcsc_footprints:C98220_R0603, F.Cu at (143.7, 86.6)
- added R44: 1KΩ, lcsc_footprints:C22548_R0603, F.Cu at (143.7, 89.0)
- added R45: 10KΩ, lcsc_footprints:C98220_R0603, F.Cu at (143.7, 91.5)
- added R46: 1KΩ, lcsc_footprints:C22548_R0603, F.Cu at (143.7, 94.0)
- added R47: 10KΩ, lcsc_footprints:C98220_R0603, F.Cu at (143.7, 96.4)
- added R48: 120Ω, lcsc_footprints:C125925_R0603, F.Cu at (143.6, 103.1)
- added R49: 100Ω, lcsc_footprints:C2906981_R0603, F.Cu at (143.7, 101.4)
- added R50: 100Ω, lcsc_footprints:C2906981_R0603, F.Cu at (143.7, 103.9)
- added R51: 100Ω, lcsc_footprints:C2906981_R0603, F.Cu at (143.7, 106.3)
- added R52: 1KΩ, lcsc_footprints:C22548_R0603, F.Cu at (147.6, 86.6)
- added R53: 10KΩ, lcsc_footprints:C98220_R0603, F.Cu at (147.6, 89.0)
- added R54: 1KΩ, lcsc_footprints:C22548_R0603, F.Cu at (147.6, 91.5)
- added R55: 10KΩ, lcsc_footprints:C98220_R0603, F.Cu at (147.6, 94.0)
- added R56: 1KΩ, lcsc_footprints:C22548_R0603, F.Cu at (147.6, 96.4)
- added R57: 10KΩ, lcsc_footprints:C98220_R0603, F.Cu at (147.6, 98.9)
- added RLED1: 0805, lcsc_footprints:C2296_LED0805-R-RD, F.Cu at (175.6, 109.6)
- added RLED2: 0805, lcsc_footprints:C2296_LED0805-R-RD, F.Cu at (175.6, 112.9)
- added RLED3: 0805, lcsc_footprints:C2296_LED0805-R-RD, F.Cu at (181.0, 103.0)
- added RLED4: 0805, lcsc_footprints:C2296_LED0805-R-RD, F.Cu at (181.0, 106.3)
- added RLED5: 0805, lcsc_footprints:C2296_LED0805-R-RD, F.Cu at (181.0, 109.6)
- added RLED6: 0805, lcsc_footprints:C2296_LED0805-R-RD, F.Cu at (181.0, 112.9)
- added RST1: RESET, Button_Switch_THT:SW_PUSH_6mm, F.Cu at (173.8, 74.8)
- added U6: ESP32-WROOM-32E(8MB), lcsc_footprints:C701342_WIFI-SMD_ESP32-WROOM-32E, F.Cu at (147.0, 74.8)
- added U7: TLP291, lcsc_footprints:C55144_SOP-4_L4_4-W2_8-P1_27-LS7_0-BR, F.Cu at (178.7, 131.0)
- added U8: CP2102N-Axx-xQFN24, Package_DFN_QFN:QFN-24-1EP_4x4mm_P0.5mm_EP2.6x2.6mm, F.Cu at (143.6, 122.3)
- added U9: ADM2587EBRWZ-REEL7, lcsc_footprints:C12081_SOIC-20_L13_0-W7_6-P1_27-LS10_3-BL, F.Cu at (186.0, 47.8)
- C1: value 100nF -> 10uF; footprint Capacitor_SMD:C_0805_2012Metric -> lcsc_footprints:C15850_C0805
- C10: value 0.1uF -> 22uF; footprint Capacitor_SMD:C_0603_1608Metric -> lcsc_footprints:C907991_C0805
- C11: value 4.7uF -> 100nF; footprint Capacitor_SMD:C_0805_2012Metric -> lcsc_footprints:C1591_C0603
- C12: footprint Capacitor_SMD:C_0603_1608Metric -> lcsc_footprints:C1591_C0603
- C13: value 100nF -> 22nF; footprint Capacitor_SMD:C_0805_2012Metric -> lcsc_footprints:C1729_C0805
- C14, C9: value 100nF -> 22nF; footprint Capacitor_SMD:C_0603_1608Metric -> lcsc_footprints:C1729_C0805
- C2: value 680 uF -> 100nF; footprint Capacitor_THT:CP_Radial_D12.5mm_P5.00mm -> lcsc_footprints:C1591_C0603
- C3: value 10uF -> 22nF; footprint Capacitor_THT:CP_Radial_D12.5mm_P5.00mm -> lcsc_footprints:C1729_C0805
- C4: value 220 uF -> 100nF; footprint Capacitor_THT:CP_Radial_D8.0mm_P3.50mm -> lcsc_footprints:C1591_C0603; moved to B.Cu
- C5: value 10uF -> 680uF; footprint Capacitor_SMD:C_1206_3216Metric -> lcsc_footprints:C48935384_CAP-TH_BD13_0-P5_00-D0_6-FD; moved to B.Cu
- C6: value 22uF -> 220uF; footprint Capacitor_SMD:C_1206_3216Metric -> lcsc_footprints:C2887273_CAP-SMD_BD6_3-L6_6-W6_6-FD; moved to B.Cu
- C7: value 100nF -> 3.3nF; footprint Capacitor_SMD:C_0603_1608Metric -> lcsc_footprints:C77036_C0603
- C8: value 100nF -> 22uF; footprint Capacitor_SMD:C_0603_1608Metric -> lcsc_footprints:C907991_C0805
- D1, L1, U1: moved to B.Cu
- D10: value BAT54JFILM -> ESD131; footprint lcsc_footprints:C86299_SOD-323_L1_8-W1_3-LS2_5-RD -> lcsc_footprints:C2939949_WLL-2-3_L0_6-W0_3-P0_36-BI
- D11: value SMAJ5.0A -> ESD131; footprint Diode_SMD:D_SMA -> lcsc_footprints:C2939949_WLL-2-3_L0_6-W0_3-P0_36-BI
- D12: value SMBJ12A -> 1N4148W; footprint lcsc_footprints:C50087775_SMB_L4_6-W3_6-LS5_3-RD -> lcsc_footprints:C917030_SOD-123_L2_8-W1_8-LS3_7-RD-1
- D13: value M7 -> SMBJ33A; footprint Diode_SMD:D_SMA -> lcsc_footprints:C353366_SMB_L4_4-W3_6-LS5_3-RD
- D3: value SS36 -> 1N4148W; footprint Diode_SMD:D_SMA -> lcsc_footprints:C917030_SOD-123_L2_8-W1_8-LS3_7-RD-1
- D4: value SS34 -> SMBJ33A; footprint Diode_SMD:D_SMA -> lcsc_footprints:C353366_SMB_L4_4-W3_6-LS5_3-RD
- D5: value PESD5V0S1UL -> SS36; footprint Diode_SMD:D_SOD-882 -> lcsc_footprints:C2922186_SMA_L4_3-W2_6-LS5_2-RD; moved to B.Cu
- D6: value ESD131 -> SS34; footprint Diode_SMD:Infineon_SG-WLL-2-3_0.58x0.28_P0.36mm -> Diode_SMD:D_SMA; moved to B.Cu
- D7: value ESD131 -> 1N4148W; footprint Diode_SMD:Infineon_SG-WLL-2-3_0.58x0.28_P0.36mm -> lcsc_footprints:C917030_SOD-123_L2_8-W1_8-LS3_7-RD-1
- D8: value SM712 -> SMBJ33A; footprint Package_TO_SOT_SMD:SOT-23 -> lcsc_footprints:C353366_SMB_L4_4-W3_6-LS5_3-RD
- D9: value BAT54JFILM -> PESD5V0S1UL; footprint lcsc_footprints:C86299_SOD-323_L1_8-W1_3-LS2_5-RD -> lcsc_footprints:C85402_SOD-882_L1_0-W0_6-RD
- F1: value 500mA -> 1.0A; footprint Fuse:Fuseholder_Clip-5x20mm_Schurter_CQM_Inline_P20.60x5.00mm_D1.00mm_Horizontal -> lcsc_footprints:C183160_F1206
- J5: value RLY PIN -> Screw_Terminal_01x02; footprint TerminalBlock_Phoenix:TerminalBlock_Phoenix_MKDS-3-3-5.08_1x03_P5.08mm_Horizontal -> TerminalBlock_Phoenix:TerminalBlock_Phoenix_MKDS-3-2-5.08_1x02_P5.08mm_Horizontal
- Q1: footprint Package_TO_SOT_SMD:SOT-23 -> lcsc_footprints:C2977534_SOT-23-3_L2_9-W1_6-P1_90-LS2_8-BR
- Q2, Q3: value MMBT3904 -> MMBT3904TT1G; footprint Package_TO_SOT_SMD:SOT-23 -> lcsc_footprints:C242260_SC-75-3_L1_6-W0_8-P1_00-LS1_6-BR
- R1, R25: value 10K -> 1KΩ; footprint Resistor_SMD:R_0805_2012Metric -> lcsc_footprints:C22548_R0603
- R10: value 20K -> 1KΩ; footprint Resistor_SMD:R_0805_2012Metric -> lcsc_footprints:C22548_R0603
- R11: value 120 -> 6.8 kΩ; footprint Resistor_SMD:R_0805_2012Metric -> lcsc_footprints:C54102246_R1206
- R12, R19: value 10K -> 4.7 kΩ; footprint Resistor_SMD:R_0805_2012Metric -> lcsc_footprints:C99782_R0603
- R13, R21: value 1K -> 2.2 kΩ; footprint Resistor_SMD:R_0805_2012Metric -> lcsc_footprints:C525570_R1206
- R14: value 680Ω -> 2.2 kΩ; footprint lcsc_footprints:C23228_R0603 -> lcsc_footprints:C525570_R1206
- R15, R23: value 10K -> 10KΩ; footprint Resistor_SMD:R_0805_2012Metric -> lcsc_footprints:C98220_R0603
- R16: value 22.1K -> 10KΩ; footprint Resistor_SMD:R_0805_2012Metric -> lcsc_footprints:C98220_R0603
- R17: value 47.5K -> 10KΩ; footprint Resistor_SMD:R_0805_2012Metric -> lcsc_footprints:C98220_R0603
- R18: value 1K -> 1KΩ; footprint Resistor_SMD:R_0805_2012Metric -> lcsc_footprints:C22548_R0603
- R2: value 10 K -> 4.7 kΩ; footprint Resistor_SMD:R_0805_2012Metric -> lcsc_footprints:C99782_R0603
- R20: value 20K -> 2.2 kΩ; footprint Resistor_SMD:R_0805_2012Metric -> lcsc_footprints:C525570_R1206
- R22: value 150Ω -> 5.1KΩ; footprint lcsc_footprints:C7065937_R0805 -> lcsc_footprints:C25905_R0402
- R24: value 100Ω -> 5.1KΩ; footprint Resistor_SMD:R_0805_2012Metric -> lcsc_footprints:C25905_R0402
- R3: value 10k -> 1KΩ; footprint Resistor_SMD:R_0805_2012Metric -> lcsc_footprints:C22548_R0603
- R4: value 10k -> 2.2 kΩ; footprint Resistor_SMD:R_0805_2012Metric -> lcsc_footprints:C525570_R1206
- R5: value 22.1K -> 2.2 kΩ; footprint Resistor_SMD:R_0805_2012Metric -> lcsc_footprints:C525570_R1206
- R6: value 10 K -> 10K
- R7: value 5.1KΩ -> 750kΩ; footprint lcsc_footprints:C25905_R0402 -> lcsc_footprints:C137684_R0603
- R8: value 5.1KΩ -> 240kΩ; footprint lcsc_footprints:C25905_R0402 -> lcsc_footprints:C137765_R0603
- R9: value 680Ω -> 1KΩ; footprint lcsc_footprints:C23228_R0603 -> lcsc_footprints:C22548_R0603; moved to B.Cu
- U2: value TLV76733DRVx -> TLP291; footprint Package_SON:WSON-6-1EP_2x2mm_P0.65mm_EP1x1.6mm_ThermalVias -> lcsc_footprints:C55144_SOP-4_L4_4-W2_8-P1_27-LS7_0-BR
- U3: value ESP32-WROOM-32E -> TLV62130RGTR; footprint RF_Module:ESP32-WROOM-32D -> lcsc_footprints:C122479_QFN-16_L3_0-W3_0-P0_50-TL-EP
- U4: value MAX485E -> TLP291; footprint Package_SO:SOIC-8_3.9x4.9mm_P1.27mm -> lcsc_footprints:C55144_SOP-4_L4_4-W2_8-P1_27-LS7_0-BR
- U5: value CP2102N-Axx-xQFN24 -> TLP291; footprint Package_DFN_QFN:QFN-24-1EP_4x4mm_P0.5mm_EP2.6x2.6mm -> lcsc_footprints:C55144_SOP-4_L4_4-W2_8-P1_27-LS7_0-BR
- moved K1 69.6 mm to (101.5, 45.5)
- moved J1 58.6 mm to (133.5, 44.1)
- moved J2 58.6 mm to (145.7, 44.1)
- moved J3 58.6 mm to (157.9, 44.1)
- moved J4 58.6 mm to (170.1, 44.1)
- moved U3 58.4 mm to (162.4, 130.8)
- moved D2 55.7 mm to (138.9, 134.6)
- moved D8 52.2 mm to (186.2, 71.4)
- moved D6 50.4 mm to (133.9, 98.8), turned to 180 degrees
- moved D7 50.1 mm to (138.3, 111.9)
- moved R14 49.9 mm to (132.8, 122.5)
- moved R8 49.0 mm to (131.9, 96.4)
- moved R7 49.0 mm to (131.9, 94.0)
- moved R24 47.2 mm to (190.4, 109.5)
- moved U5 47.2 mm to (178.7, 126.2)
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Connections:
- C1 pad 1: 24V PROTECTED -> GND
- C1 pad 2: GND -> SYS_5V
- C10 pad 1: GND -> +3V3
- C10 pad 2: +3V3 -> GND
- C11 pad 1: GND -> +3V3
- C11 pad 2: +3V3 -> GND
- C12 pad 1: GND -> EN
- C12 pad 2: Net-(U3-IO35) -> GND
- C13 pad 1: ANALOG_4_20mA -> Net-(D12-C)
- C13 pad 2: GND -> /DIN3_FIELD_GND
- C14 pad 1: GND -> Net-(D15-C)
- C14 pad 2: ANALOG_0_10V -> /DIN4_FIELD_GND
- C2 pad 1: 24V PROTECTED -> SYS_5V
- C3 pad 1: SYS_5V -> Net-(D3-C)
- C3 pad 2: GND -> /DIN1_FIELD_GND
- C4 pad 1: +5 V -> 24V PROTECTED
- C5 pad 1: +3V3 -> 24V PROTECTED
- C6 pad 1: +3V3 -> +5 V
- C7 pad 2: +3V3 -> Net-(U3-SS/TR)
- C8 pad 2: EN -> +3V3
- C9 pad 1: SYS_5V -> Net-(D7-C)
- C9 pad 2: GND -> /DIN2_FIELD_GND
- D1 pad 2: +5 V -> Net-(D1-A)
- D10 pad 1: GND -> D+
- D10 pad 2: Net-(U3-IO35) -> GND
- D11 pad 1: ANALOG_4_20mA -> D-
- D12 pad 1: Net-(D12-K) -> Net-(D12-C)
- D12 pad 2: GND -> /DIN3_FIELD_GND
- D13 pad 1: 24V PROTECTED -> Net-(D13-C)
- D13 pad 2: Net-(D13-A) -> /DIN3_FIELD_GND
- D3 pad 1: Net-(D3-K) -> Net-(D3-C)
- D3 pad 2: GND -> /DIN1_FIELD_GND
- D4 pad 1: SYS_5V -> Net-(D4-C)
- D4 pad 2: VBUS -> /DIN1_FIELD_GND
- D5 pad 1: VBUS -> Net-(D5-K)
- D6 pad 1: GND -> SYS_5V
- D6 pad 2: D+ -> +5 V
- D7 pad 1: GND -> Net-(D7-C)
- D7 pad 2: D- -> /DIN2_FIELD_GND
- D8 pad 1: RS485_B -> Net-(D8-C)
- D8 pad 2: RS485_A -> /DIN2_FIELD_GND
- D9 pad 1: +3V3 -> VBUS
- D9 pad 2: Net-(U3-IO35) -> GND
- J2 pad 1: RS485_A -> Net-(J2-0-10_V)
- J2 pad 2: RS485_B -> /DIN1_FIELD_GND
- J3 pad 1: ANALOG_4_20mA -> Net-(J3-0-10_V)
- J3 pad 2: GND -> /DIN2_FIELD_GND
- J4 pad 1: GND -> Net-(J4-0-10_V)
- J4 pad 2: GND -> /DIN3_FIELD_GND
- J5 pad 1: COM -> Net-(J5-0-10_V)
- J5 pad 2: NC -> /DIN4_FIELD_GND
- K1 pad 2: Net-(D13-A) -> Net-(D20-A)
- K1 pad 3: NO -> NO1
- K1 pad 4: COM -> COM1
- K1 pad 5: NC -> NC1
- L1 pad 1: Net-(D3-K) -> Net-(D5-K)
- Q1 pad 1: Net-(D2-K) -> Net-(D2-A)
- Q1 pad 2: Net-(D2-A) -> 24V PROTECTED
- Q1 pad 3: 24V PROTECTED -> Net-(D2-K)
- Q2 pad 2: EN -> RTS
- Q2 pad 3: RTS -> EN
- Q3 pad 2: BOOT -> DTR
- Q3 pad 3: DTR -> BOOT
- Q4 pad 3: Net-(D13-A) -> Net-(D20-A)
- R1 pad 1: GND -> +3V3
- R1 pad 2: Net-(D2-A) -> Net-(LED1-A)
- R10 pad 1: RS485_RX -> +3V3
- R10 pad 2: GND -> Net-(LED5-A)
- R11 pad 1: RS485_B -> 24V PROTECTED
- R11 pad 2: RS485_A -> Net-(LED3-+)
- R12 pad 1: RS485_RX -> DIN2
- R12 pad 2: Net-(U4-RO) -> +3V3
- R13 pad 1: ANALOG_4_20mA -> Net-(D8-C)
- R13 pad 2: Net-(U3-IO35) -> Net-(R13-Pad2)
- R14 pad 1: GND -> Net-(R13-Pad2)
- R14 pad 2: RS485_B -> Net-(D7-C)
- R15 pad 1: GND -> DTR
- R15 pad 2: RS485_DIR -> Net-(Q2-B)
- R16 pad 1: Net-(U5-VBUS) -> +3V3
- R16 pad 2: VBUS -> BOOT
- R17 pad 1: GND -> +3V3
- R17 pad 2: Net-(U5-VBUS) -> EN
- R18 pad 1: Net-(D12-K) -> +3V3
- R18 pad 2: GND -> Net-(LED6-A)
- R19 pad 1: Net-(D12-K) -> DIN3
- R19 pad 2: Net-(R19-Pad2) -> +3V3
- R2 pad 1: DTR -> DIN1
- R2 pad 2: Net-(Q2-B) -> +3V3
- R20 pad 1: Net-(R19-Pad2) -> Net-(D13-C)
- R20 pad 2: ANALOG_0_10V -> Net-(R20-Pad2)
- R21 pad 1: +3V3 -> Net-(R20-Pad2)
- R21 pad 2: Net-(U5-~{RST}) -> Net-(D12-C)
- R22 pad 1: GND -> Net-(USB-C1-CC1)
- R22 pad 2: ANALOG_4_20mA -> GND
- R23 pad 1: GND -> RTS
- R23 pad 2: ANALOG_0_10V -> Net-(Q3-B)
- R24 pad 1: Net-(Q4-G) -> Net-(USB-C1-CC2)
- R24 pad 2: RLY_CTRL -> GND
- R25 pad 1: GND -> Net-(U6-IO4)
- R25 pad 2: Net-(Q4-G) -> Net-(LED7-A)
- R3 pad 2: EN -> Net-(LED2-+)
- R4 pad 1: BOOT -> Net-(D4-C)
- R4 pad 2: +3V3 -> Net-(R4-Pad2)
- R5 pad 1: Net-(R5-Pad1) -> Net-(R4-Pad2)
- R5 pad 2: VBUS -> Net-(D3-C)
- R6 pad 1: RTS -> GND
- R6 pad 2: Net-(Q3-B) -> Net-(D2-A)
- R7 pad 1: Net-(USB-C1-CC1) -> Net-(U3-FB)
- R7 pad 2: GND -> +3V3
- R8 pad 1: Net-(USB-C1-CC2) -> Net-(U3-FB)
- R9 pad 2: RS485_A -> Net-(LED4-A)
- U1 pad 2: Net-(D3-K) -> Net-(D5-K)
- U2 pad 1: +3V3 -> Net-(D3-C)
- U2 pad 2: SYS_5V -> /DIN1_FIELD_GND
- U2 pad 4: GND -> DIN1
- U3 pad 1: GND -> Net-(L2-Pad1)
- U3 pad 10: RLY_CTRL -> SYS_5V
- U3 pad 11: unconnected-(U3-IO26-Pad11) -> SYS_5V
- U3 pad 12: RS485_DIR -> SYS_5V
- U3 pad 13: unconnected-(U3-IO14-Pad13) -> SYS_5V
- U3 pad 14: unconnected-(U3-IO12-Pad14) -> +3V3
- U3 pad 16: unconnected-(U3-IO13-Pad16) -> GND
- U3 pad 17: unconnected-(U3-NC-Pad17) -> GND
- U3 pad 2: +3V3 -> Net-(L2-Pad1)
- U3 pad 3: EN -> Net-(L2-Pad1)
- U3 pad 5: unconnected-(U3-SENSOR_VN-Pad5) -> Net-(U3-FB)
- U3 pad 6: ANALOG_0_10V -> GND
- U3 pad 7: Net-(U3-IO35) -> +3V3
- U3 pad 8: unconnected-(U3-IO32-Pad8) -> GND
- U3 pad 9: unconnected-(U3-IO33-Pad9) -> Net-(U3-SS/TR)
- U4 pad 1: Net-(U4-RO) -> Net-(D7-C)
- U4 pad 2: RS485_DIR -> /DIN2_FIELD_GND
- U4 pad 3: RS485_DIR -> GND
- U4 pad 4: RS485_TX -> DIN2
- U5 pad 1: unconnected-(U5-~{RI}/CLK-Pad1) -> Net-(D12-C)
- U5 pad 2: GND -> /DIN3_FIELD_GND
- U5 pad 3: D+ -> GND
- U5 pad 4: D- -> DIN3
- USB-C1 pad A4: Net-(R5-Pad1) -> VBUS
- USB-C1 pad A9: Net-(R5-Pad1) -> VBUS
- USB-C1 pad B4: Net-(R5-Pad1) -> VBUS
- USB-C1 pad B9: Net-(R5-Pad1) -> VBUS
