File: Industrial_IoT_Controller.kicad_sch (KiCad schematic)
At the start: 0 parts

Commit message: Updated Schematic
Parts:
- added BOOT1: BOOT, Button_Switch_THT:SW_PUSH_6mm, symbol Switch:SW_Push
- added C1, C13: 100nF, Capacitor_SMD:C_0805_2012Metric, symbol Device:C
- added C10: 0.1uF, Capacitor_SMD:C_0603_1608Metric, symbol Device:C
- added C11: 4.7uF, Capacitor_SMD:C_0805_2012Metric, symbol Device:C
- added C12, C14, C7, C8, C9: 100nF, Capacitor_SMD:C_0603_1608Metric, symbol Device:C
- added C2: 680 uF, Capacitor_THT:CP_Radial_D12.5mm_P5.00mm, symbol Device:C_Polarized
- added C3: 10uF, Capacitor_THT:CP_Radial_D12.5mm_P5.00mm, symbol Device:C
- added C4: 220 uF, Capacitor_THT:CP_Radial_D8.0mm_P3.50mm, symbol Device:C_Polarized
- added C5: 10uF, Capacitor_SMD:C_1206_3216Metric, symbol Device:C
- added C6: 22uF, Capacitor_SMD:C_1206_3216Metric, symbol Device:C
- added D1, D4: SS34, Diode_SMD:D_SMA, symbol Diode:SS34
- added D10, D9: BAT54JFILM, lcsc_footprints:C86299_SOD-323_L1_8-W1_3-LS2_5-RD, symbol lcsc_imported:BAT54JFILM
- added D11: SMAJ5.0A, Diode_SMD:D_SMA, symbol Diode:SMAJ5.0A
- added D12: SMBJ12A, lcsc_footprints:C50087775_SMB_L4_6-W3_6-LS5_3-RD, symbol lcsc_imported:SMBJ12A_C50087775
- added D13: M7, Diode_SMD:D_SMA, symbol Device:D_Small
- added D2: BZV55B15, Diode_SMD:D_MiniMELF, symbol Diode:BZV55B15
- added D3: SS36, Diode_SMD:D_SMA, symbol Diode:SS36
- added D5: PESD5V0S1UL, Diode_SMD:D_SOD-882, symbol Diode:PESD5V0S1UL
- added D6, D7: ESD131, Diode_SMD:Infineon_SG-WLL-2-3_0.58x0.28_P0.36mm, symbol Diode:ESD131-B1-W0201
- added D8: SM712, Package_TO_SOT_SMD:SOT-23, symbol Diode:SM712_SOT23
- added F1: 500mA, Fuse:Fuseholder_Clip-5x20mm_Schurter_CQM_Inline_P20.60x5.00mm_D1.00mm_Horizontal, symbol Device:Fuse
- added J1, J2, J3, J4: Screw_Terminal_01x02, TerminalBlock_Phoenix:TerminalBlock_Phoenix_MKDS-3-2-5.08_1x02_P5.08mm_Horizontal, symbol Connector:Screw_Terminal_01x02
- added J5: RLY PIN, TerminalBlock_Phoenix:TerminalBlock_Phoenix_MKDS-3-3-5.08_1x03_P5.08mm_Horizontal, symbol Connector:Screw_Terminal_01x03
- added K1: JQC-3FF/024-1ZS(551)_C2976878, lcsc_footprints:C2976878_RELAY-TH_HF_JQC-3FF, symbol lcsc_imported:JQC-3FF/024-1ZS(551)_C2976878
- added L1: 33 µH, lcsc_footprints:C177245_IND-SMD_L7_0-W6_6_FXL0630, symbol lcsc_imported:FXL0630-330-M
- added Q1: TSM2309, Package_TO_SOT_SMD:SOT-23, symbol Simulation_SPICE:PMOS
- added Q2, Q3: MMBT3904, Package_TO_SOT_SMD:SOT-23, symbol Transistor_BJT:Q_NPN_BCE
- added Q4: BSS138, lcsc_footprints:C52895_SOT-23-3_L2_9-W1_6-P1_90-LS2_8-BR, symbol lcsc_imported:BSS138_C52895
- added R1, R12, R15, R19, R23, R25: 10K, Resistor_SMD:R_0805_2012Metric, symbol Device:R
- added R10, R20: 20K, Resistor_SMD:R_0805_2012Metric, symbol Device:R
- added R11: 120, Resistor_SMD:R_0805_2012Metric, symbol Device:R
- added R13, R18, R21: 1K, Resistor_SMD:R_0805_2012Metric, symbol Device:R
- added R14, R9: 680Ω, lcsc_footprints:C23228_R0603, symbol lcsc_imported:680Ω_(6800)_±1%
- added R16, R5: 22.1K, Resistor_SMD:R_0805_2012Metric, symbol Device:R
- added R17: 47.5K, Resistor_SMD:R_0805_2012Metric, symbol Device:R
- added R2, R6: 10 K, Resistor_SMD:R_0805_2012Metric, symbol Device:R
- added R22: 150Ω, lcsc_footprints:C7065937_R0805, symbol lcsc_imported:AC0805FR-7W150RL
- added R24: 100Ω, Resistor_SMD:R_0805_2012Metric, symbol Device:R
- added R3, R4: 10k, Resistor_SMD:R_0805_2012Metric, symbol Device:R
- added R7, R8: 5.1KΩ, lcsc_footprints:C25905_R0402, symbol lcsc_imported:5_1KΩ_(5101)_±1%
- added RESET1: RESET, Button_Switch_THT:SW_PUSH_6mm, symbol Switch:SW_Push
- added U1: LM2596S-5, Package_TO_SOT_SMD:TO-263-5_TabPin3, symbol Regulator_Switching:LM2596S-5
- added U2: TLV76733DRVx, Package_SON:WSON-6-1EP_2x2mm_P0.65mm_EP1x1.6mm_ThermalVias, symbol Regulator_Linear:TLV76733DRVx
- added U3: ESP32-WROOM-32E, RF_Module:ESP32-WROOM-32D, symbol RF_Module:ESP32-WROOM-32E
- added U4: MAX485E, Package_SO:SOIC-8_3.9x4.9mm_P1.27mm, symbol Interface_UART:MAX485E
- added U5: CP2102N-Axx-xQFN24, Package_DFN_QFN:QFN-24-1EP_4x4mm_P0.5mm_EP2.6x2.6mm, symbol Interface_USB:CP2102N-Axx-xQFN24
- added USB-C1: USB_C_Receptacle_USB2.0_16P, Connector_USB:USB_C_Receptacle_HRO_TYPE-C-31-M-12, symbol Connector:USB_C_Receptacle_USB2.0_16P
Connections:
- new net: F1.1, J1.1 (A)
- new net: D2.1 (K), F1.2, Q1.1 (D)
- new net: D3.1 (K), L1.1, U1.2 (OUT)
- new net: D13.2 (A), K1.2, Q4.3 (D)
- new net: D2.2 (A), Q1.2 (G), R1.2
- new net: Q2.1 (B), R2.2
- new net: R16.1, R17.2, U5.8 (VBUS)
- new net: R21.2, U5.9 (~{RST})
- new net: C12.2, D10.2, D9.2, R13.2, U3.7 (IO35)
- new net: Q3.1 (B), R6.2
- new net: R19.2, R20.1
- new net: R12.2, U4.1 (RO)
- new net: Q4.1 (G), R24.1, R25.2
- new net: D12.1 (K), R18.1, R19.1
- new net: R5.1, USB-C1.A4 (VBUS), USB-C1.A9 (VBUS), USB-C1.B4 (VBUS), USB-C1.B9 (VBUS)
- new net: R7.1, USB-C1.A5 (CC1)
- new net: R8.1, USB-C1.B5 (CC2)
- new net +3V3: C10.2, C11.2, C5.1, C6.1, C7.2, D9.1, R21.1, R3.1, R4.2, U2.1 (OUT), U2.5 (SNS), U3.2 (VDD), U5.5 (VIO), U5.6 (VDD), U5.7 (VREGIN)
- new net +5 V: C4.1, D1.2 (A), L1.2, U1.4 (FB)
- new net 24V PROTECTED: C1.1, C2.1, D13.1 (K), K1.1, Q1.3 (S), U1.1 (VIN)
- new net ANALOG_0_10V: C14.2, R20.2, R23.2, U3.6 (IO34)
- new net ANALOG_4_20mA: C13.1, D11.1 (A1), J3.1 (4-20mA), R13.1, R22.2
- new net BOOT: BOOT1.1, Q3.2 (C), R4.1, U3.25 (IO0)
- new net COM: J5.1 (COM), K1.4
- new net D+: D6.2 (A2), U5.3 (D+), USB-C1.A6 (D+), USB-C1.B6 (D+)
- new net D-: D7.2 (A2), U5.4 (D-), USB-C1.A7 (D-), USB-C1.B7 (D-)
- new net DTR: Q3.3 (E), R2.1, U5.23 (~{DTR})
- new net EN: C8.2, Q2.2 (C), R3.2, RESET1.1, U3.3 (EN)
- new net ESP RX: U3.34 (RXD0/IO3), U5.21 (TXD)
- new net ESP TX: U3.35 (TXD0/IO1), U5.20 (RXD)
- new net GND: BOOT1.2, C1.2, C10.1, C11.1, C12.1, C13.2, C14.1, C2.2, C3.2, C4.2, C5.2, C6.2, C7.1, C8.1, C9.2, D10.1, D11.2 (A2), D12.2 (A), D3.2 (A), D5.2 (A), D6.1 (A1), D7.1 (A1), D8.3 (common), J1.2 (B), J3.2 (GND), J4.1 (0-10_V), J4.2 (GND), Q4.2 (S), R1.1, R10.2, R14.1, R15.1, R17.1, R18.2, R22.1, R23.1, R25.1, R7.2, R8.2, RESET1.2, U1.3 (GND), U1.5 (~{ON}/OFF), U2.3 (GND), U2.4 (GND), U2.7 (PAD), U3.1 (GND), U3.15 (GND), U3.38 (GND), U3.39 (GND), U4.5 (GND), U5.2 (GND), U5.25 (GND), USB-C1.A1 (GND), USB-C1.A12 (GND), USB-C1.B1 (GND), USB-C1.B12 (GND), USB-C1.SH (SHIELD)
- new net NC: J5.2 (NC), K1.5
- new net NO: J5.3 (NO), K1.3
- new net RLY_CTRL: R24.2, U3.10 (IO25)
- new net RS485_A: D8.2 (A2), J2.1 (A), R11.2, R9.2, U4.6 (A)
- new net RS485_B: D8.1 (A1), J2.2 (B), R11.1, R14.2, U4.7 (B)
- new net RS485_DIR: R15.2, U3.12 (IO27), U4.2 (~{RE}), U4.3 (DE)
- new net RS485_RX: R10.1, R12.1, U3.27 (IO16)
- new net RS485_TX: U3.28 (IO17), U4.4 (DI)
- new net RTS: Q2.3 (E), R6.1, U5.19 (~{RTS})
- new net SYS_5V: C3.1, C9.1, D1.1 (K), D4.1 (K), R9.1, U2.2 (IN), U2.6 (EN), U4.8 (VCC)
- new net VBUS: D4.2 (A), D5.1 (K), R16.2, R5.2
- no-connect marks 0 -> 29
Other:
- note added: "0-10V Sensor Input"
- note added: "24V Input"
- note added: "4-20mA Sensor"
- title: (none) -> Industrial IoT Controller

Commit message: Final Schematic
Parts:
- removed C1, C13: 100nF, Capacitor_SMD:C_0805_2012Metric, symbol Device:C
- removed C10: 0.1uF, Capacitor_SMD:C_0603_1608Metric, symbol Device:C
- removed C11: 4.7uF, Capacitor_SMD:C_0805_2012Metric, symbol Device:C
- removed C12, C14, C7, C8, C9: 100nF, Capacitor_SMD:C_0603_1608Metric, symbol Device:C
- removed C2: 680 uF, Capacitor_THT:CP_Radial_D12.5mm_P5.00mm, symbol Device:C_Polarized
- removed C3: 10uF, Capacitor_THT:CP_Radial_D12.5mm_P5.00mm, symbol Device:C
- removed C4: 220 uF, Capacitor_THT:CP_Radial_D8.0mm_P3.50mm, symbol Device:C_Polarized
- removed C5: 10uF, Capacitor_SMD:C_1206_3216Metric, symbol Device:C
- removed C6: 22uF, Capacitor_SMD:C_1206_3216Metric, symbol Device:C
- removed D11: SMAJ5.0A, Diode_SMD:D_SMA, symbol Diode:SMAJ5.0A
- removed D13: M7, Diode_SMD:D_SMA, symbol Device:D_Small
- removed D3: SS36, Diode_SMD:D_SMA, symbol Diode:SS36
- removed D5: PESD5V0S1UL, Diode_SMD:D_SOD-882, symbol Diode:PESD5V0S1UL
- removed D6, D7: ESD131, Diode_SMD:Infineon_SG-WLL-2-3_0.58x0.28_P0.36mm, symbol Diode:ESD131-B1-W0201
- removed D8: SM712, Package_TO_SOT_SMD:SOT-23, symbol Diode:SM712_SOT23
- removed F1: 500mA, Fuse:Fuseholder_Clip-5x20mm_Schurter_CQM_Inline_P20.60x5.00mm_D1.00mm_Horizontal, symbol Device:Fuse
- removed Q1: TSM2309, Package_TO_SOT_SMD:SOT-23, symbol Simulation_SPICE:PMOS
- removed Q2, Q3: MMBT3904, Package_TO_SOT_SMD:SOT-23, symbol Transistor_BJT:Q_NPN_BCE
- removed R10, R20: 20K, Resistor_SMD:R_0805_2012Metric, symbol Device:R
- removed R11: 120, Resistor_SMD:R_0805_2012Metric, symbol Device:R
- removed R12, R15, R19, R23, R25: 10K, Resistor_SMD:R_0805_2012Metric, symbol Device:R
- removed R13, R18, R21: 1K, Resistor_SMD:R_0805_2012Metric, symbol Device:R
- removed R14, R9: 680Ω, lcsc_footprints:C23228_R0603, symbol lcsc_imported:680Ω_(6800)_±1%
- removed R16, R5: 22.1K, Resistor_SMD:R_0805_2012Metric, symbol Device:R
- removed R17: 47.5K, Resistor_SMD:R_0805_2012Metric, symbol Device:R
- removed R2, R6: 10 K, Resistor_SMD:R_0805_2012Metric, symbol Device:R
- removed R24: 100Ω, Resistor_SMD:R_0805_2012Metric, symbol Device:R
- removed R3, R4: 10k, Resistor_SMD:R_0805_2012Metric, symbol Device:R
- removed U2: TLV76733DRVx, Package_SON:WSON-6-1EP_2x2mm_P0.65mm_EP1x1.6mm_ThermalVias, symbol Regulator_Linear:TLV76733DRVx
- removed U3: ESP32-WROOM-32E, RF_Module:ESP32-WROOM-32D, symbol RF_Module:ESP32-WROOM-32E
- removed U4: MAX485E, Package_SO:SOIC-8_3.9x4.9mm_P1.27mm, symbol Interface_UART:MAX485E
- added C1: 10uF, lcsc_footprints:C15850_C0805, symbol lcsc_imported:10uF_(106)_±10%_25V
- added C10, C8: 22uF, lcsc_footprints:C907991_C0805, symbol lcsc_imported:GRM21BZ71A226ME15L
- added C11, C12, C15, C16, C2, C20, C21, C25, C27, C29, C35, C37, C39, C4: 100nF, lcsc_footprints:C1591_C0603, symbol lcsc_imported:100nF_(104)_±10%_50V
- added C13, C14, C3, C9: 22nF, lcsc_footprints:C1729_C0805, symbol lcsc_imported:22nF_(223)_±10%_50V
- added C17: 4.7uF, lcsc_footprints:C1779_C0805, symbol lcsc_imported:4_7uF_(475)_±10%_25V
- added C18, C22, C30, C32: 100nF, lcsc_footprints:C1590_C0603, symbol lcsc_imported:100nF_(104)_±10%_25V
- added C19, C33: 10nF, lcsc_footprints:C100042_C0603, symbol lcsc_imported:CC0603KRX7R9BB103
- added C23, C31: 10uF, lcsc_footprints:C85713_C0603, symbol lcsc_imported:CL10A106MP8NNNC
- added C24, C26, C28, C34, C36, C38: 10uF, lcsc_footprints:C440198_C0805, symbol lcsc_imported:GRM21BR61H106KE43L
- added C5: 680uF, lcsc_footprints:C48935384_CAP-TH_BD13_0-P5_00-D0_6-FD, symbol lcsc_imported:ERG50V680M13X21
- added C6: 220uF, lcsc_footprints:C2887273_CAP-SMD_BD6_3-L6_6-W6_6-FD, symbol lcsc_imported:RVT220UF16V67RV0015
- added C7: 3.3nF, lcsc_footprints:C77036_C0603, symbol lcsc_imported:3_3nF_(332)_±5%_50V
- added D10, D11: ESD131, lcsc_footprints:C2939949_WLL-2-3_L0_6-W0_3-P0_36-BI, symbol lcsc_imported:ESD131B1W0201E6327
- added D12, D15, D3, D7: 1N4148W, lcsc_footprints:C917030_SOD-123_L2_8-W1_8-LS3_7-RD-1, symbol lcsc_imported:1N4148W_C917030
- added D13, D16, D4, D8: SMBJ33A, lcsc_footprints:C353366_SMB_L4_4-W3_6-LS5_3-RD, symbol lcsc_imported:SMBJ33A_C353366
- added D18: SMAJ5.0A, lcsc_footprints:C83329_SMA_L4_3-W2_6-LS5_2-RD, symbol lcsc_imported:SMAJ5_0A-C83329
- added D20, D21, D22, D24, D25, D26: SS14, lcsc_footprints:C2480_SMA_L4_2-W2_6-LS5_0-RD_1, symbol lcsc_imported:SS14
- added D23: SM712, Package_TO_SOT_SMD:SOT-23, symbol Diode:SM712_SOT23
- added D5: SS36, lcsc_footprints:C2922186_SMA_L4_3-W2_6-LS5_2-RD, symbol lcsc_imported:SS36_C2922186
- added D9: PESD5V0S1UL, lcsc_footprints:C85402_SOD-882_L1_0-W0_6-RD, symbol lcsc_imported:PESD5V0S1UL,315
- added F1: 1.0A, lcsc_footprints:C183160_F1206, symbol lcsc_imported:S1206-S-1_0A
- added F2: 500 mA, lcsc_footprints:C163512_F1206, symbol lcsc_imported:1206L050YR
- added F3, F4, F5, F6: SMD0805-010-60V, lcsc_footprints:C6851463_F0805, symbol lcsc_imported:SMD0805-010-60V
- added J10, J12, J13, J14, J15, J9: RLY PIN, TerminalBlock_Phoenix:TerminalBlock_Phoenix_MKDS-3-3-5.08_1x03_P5.08mm_Horizontal, symbol Connector:Screw_Terminal_01x03
- added J11: Short Circuit Cap, lcsc_footprints:C5305_FL_001, symbol lcsc_imported:2_54短路帽开口
- added J3, J4, J5: Screw_Terminal_01x02, TerminalBlock_Phoenix:TerminalBlock_Phoenix_MKDS-3-2-5.08_1x02_P5.08mm_Horizontal, symbol Connector:Screw_Terminal_01x02
- added JP1: RS485_TERM, lcsc_footprints:C32713268_HDR-TH_2P-P2_54-V-M-3, symbol lcsc_imported:HX_PZ2_54-1X2P_ZZ
- added K2, K3, K4, K5, K6: JQC-3FF/024-1ZS(551)_C2976878, lcsc_footprints:C2976878_RELAY-TH_HF_JQC-3FF, symbol lcsc_imported:JQC-3FF/024-1ZS(551)_C2976878
- added L2: 2.2 uH, lcsc_footprints:C53198556_IND-SMD_L4_1-W4_1_ASFPIG4020, symbol lcsc_imported:GXTC0420-2R2-MT
- added L3, L4: 600Ω±25% @100MHz, lcsc_footprints:C85833_L0603, symbol lcsc_imported:600Ω±25%_@100MHz
- added LED1, LED2, LED5, LED6, LED8, RLED1, RLED2, RLED3, RLED4, RLED5, RLED6: 0805, lcsc_footprints:C2296_LED0805-R-RD, symbol lcsc_imported:0805
- added LED3: YLED0805R, lcsc_footprints:C19171391_LED0805-R-RD_RED, symbol lcsc_imported:YLED0805R
- added LED4, LED7: XL-2012UBC, lcsc_footprints:C965817_LED0805-RD, symbol lcsc_imported:XL-2012UBC
- added Q1: TSM2309, lcsc_footprints:C2977534_SOT-23-3_L2_9-W1_6-P1_90-LS2_8-BR, symbol lcsc_imported:TSM2309CX_RFG
- added Q2, Q3: MMBT3904TT1G, lcsc_footprints:C242260_SC-75-3_L1_6-W0_8-P1_00-LS1_6-BR, symbol lcsc_imported:MMBT3904TT1G
- added Q5, Q6, Q7, Q8, Q9: BSS138, lcsc_footprints:C52895_SOT-23-3_L2_9-W1_6-P1_90-LS2_8-BR, symbol lcsc_imported:BSS138_C52895
- added R1, R10, R18, R25, R26, R3, R30, R33, R37, R42, R44, R46, R52, R54, R56, R9: 1KΩ, lcsc_footprints:C22548_R0603, symbol lcsc_imported:1KΩ_(1001)_±1%
- added R11: 6.8 kΩ, lcsc_footprints:C54102246_R1206, symbol lcsc_imported:FRP1206F6801TS
- added R12, R19, R2, R27: 4.7 kΩ, lcsc_footprints:C99782_R0603, symbol lcsc_imported:RC0603FR-074K7L
- added R13, R14, R20, R21, R28, R29, R4, R5: 2.2 kΩ, lcsc_footprints:C525570_R1206, symbol lcsc_imported:ESR18EZPF2201
- added R15, R16, R17, R23, R34, R38, R43, R45, R47, R53, R55, R57: 10KΩ, lcsc_footprints:C98220_R0603, symbol lcsc_imported:RC0603FR-0710KL
- added R31: 22.1KΩ, lcsc_footprints:C2960862_R0603, symbol lcsc_imported:FRC0603F2212TS
- added R32: 47.KΩ, lcsc_footprints:C403243_R0603, symbol lcsc_imported:ERJ3EKF4752V
- added R35: 20KΩ, lcsc_footprints:C2907011_R0603, symbol lcsc_imported:FRC0603F2002TS
- added R39, R40, R41, R49, R50, R51: 100Ω, lcsc_footprints:C2906981_R0603, symbol lcsc_imported:FRC0603F1000TS
- added R48: 120Ω, lcsc_footprints:C125925_R0603, symbol lcsc_imported:AC0603FR-07120RL
- added R7: 750kΩ, lcsc_footprints:C137684_R0603, symbol lcsc_imported:RC0603FR-07750KL
- added R8: 240kΩ, lcsc_footprints:C137765_R0603, symbol lcsc_imported:RC0603FR-07240KL
- added U2, U4, U5, U7: TLP291, lcsc_footprints:C55144_SOP-4_L4_4-W2_8-P1_27-LS7_0-BR, symbol lcsc_imported:TLP291(GB-TP,SE(T
- added U3: TLV62130RGTR, lcsc_footprints:C122479_QFN-16_L3_0-W3_0-P0_50-TL-EP, symbol lcsc_imported:TLV62130RGTR
- added U6: ESP32-WROOM-32E(8MB), lcsc_footprints:C701342_WIFI-SMD_ESP32-WROOM-32E, symbol lcsc_imported:ESP32-WROOM-32E(8MB)
- added U9: ADM2587EBRWZ-REEL7, lcsc_footprints:C12081_SOIC-20_L13_0-W7_6-P1_27-LS10_3-BL, symbol lcsc_imported:ADM2587EBRWZ-REEL7
- renumbered D4 to D1, D9 to D14, D10 to D17, D12 to D19, D1 to D6, J3 to J6, J4 to J7, J5 to J8, R7 to R22, R8 to R24, R22 to R36, R1 to R6, RESET1 to RST1, U5 to U8
Connections:
- net +3V3: now also C10.1, C11.1, C16.1, C17.1, C18.2, C19.2, C22.1, C23.1, C8.2, L2.2, R1.1, R10.1, R12.2, R16.1, R17.1, R18.1, R19.2, R2.2, R26.1, R27.2, R3.1, R37.2, R7.2, U3.14 (VOS), U3.7 (FSW), U6.2 (3V3), U9.2 (VCC), U9.8 (VCC)
- net +5 V: now also C6.1
- net 24V PROTECTED: now also C24.1, C25.1, C26.1, C27.1, C28.1, C29.1, C34.1, C35.1, C36.1, C37.1, C38.1, C39.1, C4.1, C5.1, D20.1 (K), D21.1 (K), D22.1 (K), D24.1 (K), D25.1 (K), D26.1 (K), K2.1, K3.1, K4.1, K5.1, K6.1, Q1.2 (S), R11.1
- net ANALOG_0_10V: now also C21.1, R35.2, R38.1, U6.6 (IO34)
- net ANALOG_4_20mA: now also C20.1, D18.1 (C), R30.2
- net BOOT: now also Q3.3 (C), R16.2, U6.25 (IO0)
- net D+: now also D10.1
- net D-: now also D11.1
- net DTR: now also Q3.2 (E), R15.1
- net EN: now also C12.1, Q2.3 (C), R17.2, U6.3 (EN)
- net ESP RX: now also U6.34 (RXD0)
- net ESP TX: now also U6.35 (TXD0)
- net GND: now also D17.2, C1.1, C10.2, C11.2, C12.2, C15.2, C16.2, C17.2, C18.1, C19.1, C2.2, C20.2, C21.2, C22.2, C23.2, C4.2, C5.2, C6.2, C7.1, C8.1, D10.2, D11.2, D18.2 (A), D5.2 (A), D9.2 (A), LED2.2 (-), LED3.2 (-), LED4.1 (K), LED7.1 (K), Q5.2 (S), Q6.2 (S), Q7.2 (S), Q8.2 (S), Q9.2 (S), R32.2, R38.2, R43.2, R45.2, R47.2, R53.2, R55.2, R57.2, R8.2, RLED1.2 (-), RLED2.2 (-), RLED3.2 (-), RLED4.2 (-), RLED5.2 (-), RLED6.2 (-), U2.3, U3.15 (PGND), U3.16 (PGND), U3.17 (EXP), U3.6 (AGND), U3.8 (DEF), U4.3, U5.3, U6.15 (GND), U7.3, U9.1 (GND1), U9.10 (GND1), U9.3 (GND1), U9.9 (GND1); no longer D17.1, J7.1 (0-10_V)
- net RS485_A: now also D23.1 (A1), J12.1 (Pin_1), R48.1, U9.13 (Y), U9.18 (A); no longer J2.1 (A)
- net RS485_B: now also D23.2 (A2), J12.2 (Pin_2), JP1.2, U9.15 (Z), U9.17 (B); no longer J2.2 (B)
- net RS485_DIR: now also U6.12 (IO27), U9.5 (RE#), U9.6 (DE)
- net RS485_RX: now also U6.27 (IO16), U9.4 (RXD)
- net RS485_TX: now also U6.28 (IO17), U9.7 (TXD)
- net RTS: now also Q2.2 (E), R23.1
- net SYS_5V: now also C1.2, C2.1, R9.1, U3.10 (AVIN), U3.11 (PVIN), U3.12 (PVIN), U3.13 (EN)
- net VBUS: now also USB-C1.A4 (VBUS), USB-C1.A9 (VBUS), USB-C1.B4 (VBUS), USB-C1.B9 (VBUS), D9.1 (C), F2.1, R31.2; no longer D1.2 (A)
- net at J1.1 (Pin_1): now also F1.1
- net at D2.1 (K): now also F1.2, Q1.3 (D)
- net at L1.1, U1.2 (OUT): now also D5.1 (K)
- net at K1.2, Q4.3 (D): now also C24.2, C25.2, D20.2 (A)
- net at D2.2 (A), R6.2: now also Q1.1 (G)
- net at U8.8 (VBUS): now also R31.1, R32.1
- net at U8.9 (~{RST}): now also R37.1
- net 4_20mA: now reaches D14.2
- net 4_20mA: now also D17.1, C15.1, R30.1, U6.7 (IO35); no longer D17.2
- net at Q4.1 (G): now also R39.2, R43.1
- net at D19.1 (K): now also R33.2, R34.1
- net COM renamed COM1
- net NC renamed NC1
- net NO renamed NO1
- new net: LED3.1 (+), R11.2
- new net: F3.1, J2.1 (Pin_1)
- new net: D4.1 (C), F3.2, R4.1
- new net: F6.1, J5.1 (Pin_1)
- new net: R46.1, RLED3.1 (+)
- new net: R42.1, RLED1.1 (+)
- new net: C34.2, C35.2, D24.2 (A), K4.2, Q7.3 (D)
- new net: Q8.1 (G), R50.2, R55.1
- new net: LED5.1 (+), R10.2
- new net: R56.1, RLED6.1 (+)
- new net: C3.1, D3.1 (C), R5.2, U2.1
- new net: Q6.1 (G), R41.2, R47.1
- new net: C14.1, D15.1 (C), R29.2, U7.1
- new net: C28.2, C29.2, D22.2 (A), K3.2, Q6.3 (D)
- new net: C38.2, C39.2, D26.2 (A), K6.2, Q9.3 (D)
- new net: D13.1 (C), F5.2, R20.1
- new net: C36.2, C37.2, D25.2 (A), K5.2, Q8.3 (D)
- new net: C13.1, D12.1 (C), R21.2, U5.1
- new net: R34.2, R35.1
- new net: F4.1, J3.1 (Pin_1)
- new net: D8.1 (C), F4.2, R13.1
- new net: JP1.1, R48.2
- new net: L2.1, U3.1 (SW), U3.2 (SW), U3.3 (SW)
- new net: LED8.1 (+), R26.2
- new net: LED2.1 (+), R3.2
- new net: LED6.1 (+), R18.2
- new net: Q3.1 (B), R23.2
- new net: R54.1, RLED5.1 (+)
- new net: R52.1, RLED4.1 (+)
- new net: D16.1 (C), F6.2, R28.1
- new net: LED4.2 (A), R9.2
- new net: R13.2, R14.1
- new net: C9.1, D7.1 (C), R14.2, U4.1
- new net: R44.1, RLED2.1 (+)
- new net: R7.1, R8.1, U3.5 (FB)
- new net: U6.1 (GND), U6.38 (GND), U6.39 (GND)
- new net: R25.1, U6.26 (IO4)
- new net: Q7.1 (G), R49.2, R53.1
- new net: D1.2 (A), F2.2
- new net: J7.1 (Pin_1), R33.1
- new net: C26.2, C27.2, D21.2 (A), K2.2, Q5.3 (D)
- new net: R4.2, R5.1
- new net: LED1.1 (+), R1.2
- new net: Q5.1 (G), R40.2, R45.1
- new net: R28.2, R29.1
- new net: Q9.1 (G), R51.2, R57.1
- new net: F5.1, J4.1 (Pin_1)
- new net: C7.2, U3.9 (SS/TR)
- new net: R20.2, R21.1
- new net: LED7.2 (A), R25.2
- new net: Q2.1 (B), R15.2
- new net COM2: J9.1 (Pin_1), K2.4
- new net COM3: J10.1 (Pin_1), K3.4
- new net COM4: J13.1 (Pin_1), K4.4
- new net COM5: J14.1 (Pin_1), K5.4
- new net COM6: J15.1 (Pin_1), K6.4
- new net DIN1: LED1.2 (-), R2.1, U2.4, U6.8 (IO32)
- new net DIN1_FIELD_GND: C3.2, D3.2 (A), D4.2 (A), J2.2 (Pin_2), U2.2
- new net DIN2: LED5.2 (-), R12.1, U4.4, U6.9 (IO33)
- new net DIN2_FIELD_GND: C9.2, D7.2 (A), D8.2 (A), J3.2 (Pin_2), U4.2
- new net DIN3: LED6.2 (-), R19.1, U5.4, U6.4 (SENSOR_VP)
- new net DIN3_FIELD_GND: C13.2, D12.2 (A), D13.2 (A), J4.2 (Pin_2), U5.2
- new net DIN4: LED8.2 (-), R27.1, U6.5 (SENSOR_VN), U7.4
- new net DIN4_FIELD_GND: C14.2, D15.2 (A), D16.2 (A), J5.2 (Pin_2), U7.2
- new net GND_ISO_PWR: C30.2, C31.2, L4.1, U9.11 (GND2), U9.14 (GND2)
- new net NC2: J9.2 (Pin_2), K2.5
- new net NC3: J10.2 (Pin_2), K3.5
- new net NC4: J13.2 (Pin_2), K4.5
- new net NC5: J14.2 (Pin_2), K5.5
- new net NC6: J15.2 (Pin_2), K6.5
- new net NO2: J9.3 (Pin_3), K2.3
- new net NO3: J10.3 (Pin_3), K3.3
- new net NO4: J13.3 (Pin_3), K4.3
- new net NO5: J14.3 (Pin_3), K5.3
- new net NO6: J15.3 (Pin_3), K6.3
- new net RLY1_CTRL: R39.1, R42.2, U6.30 (IO18)
- new net RLY2_CTRL: R40.1, R44.2, U6.31 (IO19)
- new net RLY3_CTRL: R41.1, R46.2, U6.33 (IO21)
- new net RLY4_CTRL: R49.1, R52.2, U6.36 (IO22)
- new net RLY5_CTRL: R50.1, R54.2, U6.37 (IO23)
- new net RLY6_CTRL: R51.1, R56.2, U6.11 (IO26)
- new net RS485_ISO_GND: C32.2, C33.2, D23.3 (common), J12.3 (Pin_3), L4.2, U9.16 (GND2), U9.20 (GND2)
- new net VISOIN: C32.1, C33.1, L3.2, U9.19 (VISOIN)
- new net VISO_FILT: C30.1, C31.1, L3.1, U9.12 (VISOOUT)
- no-connect marks 29 -> 28
Other:
- note added: "24VDC Input"
- note added: "24VDC to 5VDC Converter"
- note added: "4-20mA Sensor Input"
- note added: "5VDC to 3.3VDC Converter"
- note added: "Auto Programming Mode"
- note added: "CP2102N USB to UART"
- note added: "ESPESP32-WROOM-32E(8MB)"
- note added: "Isolated Input 1"
- note added: "Isolated Input 2"
- note added: "Isolated Input 3"
- note added: "Isolated Input 4"
- note added: "Isolated RS485"
- note added: "Relay1"
- note added: "Relay2"
- note added: "Relay3"
- note added: "Relay4"
- note added: "Relay5"
- note added: "Relay6"
- note added: "USB-C Connector"
- note removed: "24V Input"
- note removed: "4-20mA Sensor"
- moved on the sheet: D1, D14, D17, D19, D2, D6, J1, J6, J7, J8, K1, Q4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
